Commit message: Update: xacro robot description is now caught up with new robot

File: src/robot_description/description/component_macros.xacro (robot description, xacro)
@@ -2,5 +2,5 @@
 <robot xmlns:xacro="http://ros.org/wiki/xacro">
 <!-- basic building blocks -->
-<xacro:macro name="box_link" params="name mass x y z material:=red">
+<xacro:macro name="box_link" params="name mass x y z material:=red origin_position:='0 0 0' origin_orientation:='0 0 0'">
     <link name="${name}">
         <inertial>
@@ -9,4 +9,5 @@
                      iyy="${(1/12) * mass * (x*x+z*z)}" iyz="0.0"
                      izz="${(1/12) * mass * (x*x+y*y)}" />
+            <origin xyz="${origin_position}" rpy="${origin_orientation}"/>
         </inertial>
         <visual>
@@ -15,4 +16,5 @@
             </geometry>
             <material name="${material}"/>
+            <origin xyz="${origin_position}" rpy="${origin_orientation}"/>
         </visual>
         <collision>
@@ -20,8 +22,9 @@
                 <box size="${x} ${y} ${z}"/>
             </geometry>
-        </collision>
-    </link>
-</xacro:macro>
-<xacro:macro name="cylinder_link" params="name mass radius length material:=red">
+            <origin xyz="${origin_position}" rpy="${origin_orientation}"/>
+        </collision>
+    </link>
+</xacro:macro>
+<xacro:macro name="cylinder_link" params="name mass radius length material:=red origin_position:='0 0 0' origin_orientation:='0 0 0'">
     <link name="${name}">
         <inertial>
@@ -30,4 +33,5 @@
                      iyy="${(1/12) * mass * (3*radius*radius + length*length)}" iyz="0.0"
                      izz="${(1/2) * mass * (radius*radius)}" />
+            <origin xyz="${origin_position}" rpy="${origin_orientation}"/>
         </inertial>
         <visual>
@@ -36,4 +40,5 @@
             </geometry>
             <material name="${material}"/>
+            <origin xyz="${origin_position}" rpy="${origin_orientation}"/>
         </visual>
         <collision>
@@ -41,8 +46,9 @@
                 <cylinder radius="${radius}" length="${length}"/>
             </geometry>
-        </collision>
-    </link>
-</xacro:macro>
-<xacro:macro name="ball_link" params="name mass radius material:=red">
+            <origin xyz="${origin_position}" rpy="${origin_orientation}"/>
+        </collision>
+    </link>
+</xacro:macro>
+<xacro:macro name="ball_link" params="name mass radius material:=red origin_position:='0 0 0' origin_orientation:='0 0 0'">
     <link name="${name}">
         <inertial>
@@ -52,4 +58,5 @@
                 iyy="0.002" iyz="0.0"
                 izz="0.002"/>
+            <origin xyz="${origin_position}" rpy="${origin_orientation}"/>
         </inertial>
         <visual>
@@ -58,4 +65,5 @@
             </geometry>
             <material name="${material}"/>
+            <origin xyz="${origin_position}" rpy="${origin_orientation}"/>
         </visual>
         <collision>
@@ -63,4 +71,5 @@
                 <sphere radius="${radius}"/>
             </geometry>
+            <origin xyz="${origin_position}" rpy="${origin_orientation}"/>
         </collision>
     </link>
@@ -75,20 +84,20 @@
         </inertial> -->
         <visual>
-            <origin xyz="${origin_position}" rpy="${origin_orientation}"/>
-            <geometry>
-                <mesh filename="package://${package}/${file}" scale="${scale} ${scale} ${scale}"/>
-            </geometry>
-            <material name="${material}"/>
-        </visual>
-        <collision>
-            <origin xyz="${origin_position}" rpy="${origin_orientation}"/>
-            <geometry>
-                <mesh filename="package://${package}/${file}" scale="${scale} ${scale} ${scale}"/>
-            </geometry>
+            <geometry>
+                <mesh filename="file://$(find ${package})/${file}" scale="${scale} ${scale} ${scale}"/>
+            </geometry>
+            <material name="${material}"/>
+            <origin xyz="${origin_position}" rpy="${origin_orientation}"/>
+        </visual>
+        <collision>
+            <geometry>
+                <mesh filename="file://$(find ${package})/${file}" scale="${scale} ${scale} ${scale}"/>
+            </geometry>
+            <origin xyz="${origin_position}" rpy="${origin_orientation}"/>
         </collision>
     </link>
 </xacro:macro>
 <xacro:macro name="fixed_joint" params="name parent child origin_position:='0 0 0' origin_orientation:='0 0 0'">
-    <joint name="${name}_joint" type="fixed">
+    <joint name="${name}" type="fixed">
         <parent link="${parent}"/>
         <child link="${child}"/>
@@ -97,5 +106,5 @@
 </xacro:macro>
 <xacro:macro name="continuous_joint" params="name parent child origin_position:='0 0 0' origin_orientation:='0 0 0' axis='0 0 0'">
-    <joint name="${name}_joint" type="continuous">
+    <joint name="${name}" type="continuous">
         <parent link="${parent}"/>
         <child link="${child}"/>
@@ -105,5 +114,5 @@
 </xacro:macro>
 <xacro:macro name="floating_joint" params="name parent child origin_position:='0 0 0' origin_orientation:='0 0 0'">
-    <joint name="${name}_joint" type="floating">
+    <joint name="${name}" type="floating">
         <parent link="${parent}"/>
         <child link="${child}"/>

File: src/robot_description/description/frame.xacro (robot description, xacro)
@@ -4,42 +4,132 @@
     <link name="base_link"/>
     <link name="base_footprint"/>
-    <xacro:fixed_joint name="base_footprint" parent="base_link" child="base_footprint"/>
+    <xacro:fixed_joint name="base_link_to_base_footprint" parent="base_link" child="base_footprint"/>
 </xacro:macro>
-<xacro:macro name="robot_chassis">
-    <xacro:mesh_link name="baseplate" package="robot_description" file="description/meshes/orp_baseplate.stl"/>
+<xacro:macro name="robot_description">
+    <xacro:chassis/>
+    <xacro:power_source/>
+    <xacro:motors_and_wheels/>
+    <xacro:sensors_and_accurators/>
+</xacro:macro>
+<!-- orp baseplate and adapters -->
+<xacro:macro name="chassis">
+    <xacro:mesh_link name="baseplate" package="robot_description" file="description/meshes/orp_baseplate.stl"
+                     origin_orientation="1.5708 0 1.5708"/>
     <xacro:fixed_joint name="base_link_to_baseplate" parent="base_link" child="baseplate"
-                       origin_position="0 0 0" origin_orientation="1.5708 0 0"/>
-    <xacro:mesh_link name="left_motor_bracket" package="robot_description" file="description/meshes/orp_jga25-371_motor_adapter.stl"/>
+                       origin_position="0 0 0"/>
+    <xacro:mesh_link name="rpi_adapter" package="robot_description" file="description/meshes/orp_rpi4b_adapter.stl"
+                     origin_orientation="1.5708 0 1.5708"/>
+    <xacro:fixed_joint name="baseplate_to_rpi_adapter" parent="baseplate" child="rpi_adapter"
+                       origin_position="0.010 0 0.005"/>
+    <xacro:mesh_link name="left_motor_bracket" package="robot_description" file="description/meshes/orp_jga25-371_motor_adapter.stl"
+                     origin_orientation="-1.5708 0 0"/>
     <xacro:fixed_joint name="baseplate_to_left_motor_bracket" parent="baseplate" child="left_motor_bracket"
-                       origin_position="0.080 0 0" origin_orientation="0 -1.5708 3.1415"/>
-    <xacro:mesh_link name="right_motor_bracket" package="robot_description" file="description/meshes/orp_jga25-371_motor_adapter.stl"/>
+                       origin_position="0 0.080 0"/>
+    <xacro:mesh_link name="right_motor_bracket" package="robot_description" file="description/meshes/orp_jga25-371_motor_adapter.stl"
+                     origin_orientation="-1.5708 0 3.1415"/>
     <xacro:fixed_joint name="baseplate_to_right_motor_bracket" parent="baseplate" child="right_motor_bracket"
-                       origin_position="-0.080 0 0" origin_orientation="0 1.5708 3.1415"/>
-    <xacro:mesh_link name="front_caster_adapter" package="robot_description" file="description/meshes/orp_caster_wheel_adapter.stl"/>
+                       origin_position="0 -0.080 0"/>
+    <xacro:mesh_link name="front_caster_adapter" package="robot_description" file="description/meshes/orp_caster_wheel_adapter.stl"
+                     origin_orientation="-1.5708 0 1.5708"/>
     <xacro:fixed_joint name="baseplate_to_front_caster_adapter" parent="baseplate" child="front_caster_adapter"
-                       origin_position="0 0 0.080" origin_orientation="3.1415 0 0"/>
-    <xacro:mesh_link name="back_caster_adapter" package="robot_description" file="description/meshes/orp_caster_wheel_adapter.stl"/>
+                       origin_position="0.080 0 0"/>
+    <xacro:mesh_link name="back_caster_adapter" package="robot_description" file="description/meshes/orp_caster_wheel_adapter.stl"
+                     origin_orientation="-1.5708 0 1.5708"/>
     <xacro:fixed_joint name="baseplate_to_back_caster_adapter" parent="baseplate" child="back_caster_adapter"
-                       origin_position="0 0 -0.080" origin_orientation="3.1415 0 0"/>
+                       origin_position="-0.080 0 0"/>
+    <xacro:mesh_link name="servo_adapter" package="robot_description" file="description/meshes/orp_servo_adapter.stl"
+                     origin_orientation="1.5708 0 1.5708"/>
+    <xacro:fixed_joint name="baseplate_to_servo_adapter" parent="baseplate" child="servo_adapter"
+                       origin_position="0.100 0 0.0075"/>
+    <xacro:mesh_link name="camera_adapter" package="robot_description" file="description/meshes/orp_camera_adapter.stl"
+                     origin_orientation="1.5708 0 1.5708"/>
+    <xacro:fixed_joint name="baseplate_to_camera_adapter" parent="baseplate" child="camera_adapter"
+                       origin_position="0.0635 0.060 0.005"/>
+    <xacro:mesh_link name="spacer_1" package="robot_description" file="description/meshes/orp_spacer.stl"
+                     origin_orientation="1.5708 0 0"/>
+    <xacro:fixed_joint name="baseplate_to_spacer_1" parent="baseplate" child="spacer_1"
+                       origin_position="-0.040 -0.080 0.005"/>
+    <xacro:mesh_link name="spacer_2" package="robot_description" file="description/meshes/orp_spacer.stl"
+                     origin_orientation="1.5708 0 0"/>
+    <xacro:fixed_joint name="baseplate_to_spacer_2" parent="baseplate" child="spacer_2"
+                       origin_position="-0.040 0 0.005"/>
+    <xacro:mesh_link name="spacer_3" package="robot_description" file="description/meshes/orp_spacer.stl"
+                     origin_orientation="1.5708 0 0"/>
+    <xacro:fixed_joint name="baseplate_to_spacer_3" parent="baseplate" child="spacer_3"
+                       origin_position="0.060 0 0.005"/>
+    <xacro:mesh_link name="spacer_4" package="robot_description" file="description/meshes/orp_spacer.stl"
+                     origin_orientation="1.5708 0 0"/>
+    <xacro:fixed_joint name="baseplate_to_spacer_4" parent="baseplate" child="spacer_4"
+                       origin_position="0.060 -0.080 0.005"/>
+    <xacro:mesh_link name="lidar_adapter" package="robot_description" file="description/meshes/orp_lidar.stl"
+                     origin_orientation="1.5708 0 3.1415"/>
+    <xacro:fixed_joint name="baseplate_to_lidar_adapter" parent="baseplate" child="lidar_adapter"
+                       origin_position="0.0085 -0.040 0.1075"/>
 </xacro:macro>
+<!-- battery model (mainly included weight and visual) -->
+<xacro:macro name="power_source">
+    <xacro:mesh_link name="battery_base" package="robot_description" file="description/meshes/orp_battery_base.stl"
+                     origin_orientation="0 -1.5708 3.1415"/>
+    <xacro:fixed_joint name="baseplate_to_battery_base" parent="baseplate" child="battery_base"
+                       origin_position="-0.059 0.035 0.020"/>
+    <xacro:mesh_link name="battery_top" package="robot_description" file="description/meshes/orp_battery_top.stl"
+                     origin_orientation="0 -1.5708 3.1415"/>
+    <xacro:fixed_joint name="baseplate_to_battery_top" parent="battery_base" child="battery_top"
+                       origin_position="0 0.030 0"/>
+    <xacro:mesh_link name="battery_bottom" package="robot_description" file="description/meshes/orp_battery_bottom.stl"
+                     origin_orientation="0 -1.5708 3.1415"/>
+    <xacro:fixed_joint name="baseplate_to_battery_bottom" parent="battery_base" child="battery_bottom"
+                       origin_position="0 -0.020 0"/>
+    <xacro:mesh_link name="battery_bms_charger_cover" package="robot_description" file="description/meshes/orp_battery_bms_charger_cover.stl"
+                     origin_orientation="0 -1.5708 3.1415"/>
+    <xacro:fixed_joint name="baseplate_to_battery_bms_charger_cover" parent="battery_base" child="battery_bms_charger_cover"
+                       origin_position="0 0 -0.053"/>
+</xacro:macro>
+<!-- wheels are important here they are used by ros2_control, motors are just visual -->
 <xacro:macro name="motors_and_wheels">
-    <xacro:cylinder_link name="left_motor" mass="20" radius="0.010" length="0.050"/>
+    <xacro:cylinder_link name="left_motor" mass="20" radius="0.010" length="0.050"
+                         origin_orientation="1.5708 0 0"/>
     <xacro:fixed_joint name="left_motor_bracket_to_left_motor" parent="left_motor_bracket" child="left_motor"
-                       origin_position="0 0.020 -0.030" origin_orientation="0 0 0"/>
-    <xacro:cylinder_link name="right_motor" mass="20" radius="0.010" length="0.050"/>
+                       origin_position="0 -0.025 -0.0175"/>
+    <xacro:cylinder_link name="left_wheel" mass="20" radius="0.025" length="0.020"
+                         origin_orientation="1.5708 0 0"/>
+    <xacro:continuous_joint name="left_motor_bracket_to_left_wheel" parent="left_motor_bracket" child="left_wheel"
+                            origin_position="0 0.025 -0.0175" axis="0 1 0"/>
+    <xacro:cylinder_link name="right_motor" mass="20" radius="0.010" length="0.050"
+                     origin_orientation="1.5708 0 0"/>
     <xacro:fixed_joint name="right_motor_bracket_to_right_motor" parent="right_motor_bracket" child="right_motor"
-                       origin_position="0 0.020 -0.030" origin_orientation="0 0 0"/>
-    <xacro:cylinder_link name="left_wheel" mass="20" radius="0.025" length="0.020"/>
-    <xacro:continuous_joint name="left_motor_bracket_to_left_wheel" parent="left_motor_bracket" child="left_wheel"
-                            origin_position="0 0.020 0.025" origin_orientation="0 0 0" axis="0 0 1"/>
-    <xacro:cylinder_link name="right_wheel" mass="20" radius="0.025" length="0.020"/>
+                       origin_position="0 0.025 -0.0175"/>
+    <xacro:cylinder_link name="right_wheel" mass="20" radius="0.025" length="0.020"
+                         origin_orientation="1.5708 0 0"/>
     <xacro:continuous_joint name="right_motor_bracket_to_right_wheel" parent="right_motor_bracket" child="right_wheel"
-                            origin_position="0 0.020 0.025" origin_orientation="0 0 0" axis="0 0 1"/>
+                            origin_position="0 -0.025 -0.0175" axis="0 1 0"/>
     <xacro:ball_link name="front_caster_wheel" mass="1" radius="0.010"/>
-    <xacro:floating_joint name="front_caster_adapter_to_front_caster_wheel" parent="front_caster_adapter" child="front_caster_wheel"
-                        origin_position="0 0.035 0" origin_orientation="0 0 0"/>
+    <xacro:fixed_joint name="front_caster_adapter_to_front_caster_wheel" parent="front_caster_adapter" child="front_caster_wheel"
+                       origin_position="0 0 -0.035"/>
     <xacro:ball_link name="back_caster_wheel" mass="1" radius="0.010"/>
-    <xacro:continuous_joint name="back_caster_adapter_to_back_caster_wheel" parent="back_caster_adapter" child="back_caster_wheel"
-                        origin_position="0 0.035 0" origin_orientation="0 0 0"/>
+    <xacro:fixed_joint name="back_caster_adapter_to_back_caster_wheel" parent="back_caster_adapter" child="back_caster_wheel"
+                       origin_position="0 0 -0.035"/>
+</xacro:macro>
+<!-- representation of servo, ultrasonic, camera and lidar, gazebo plugins reference these -->
+<xacro:macro name="sensors_and_accurators">
+    <xacro:box_link name="servo" mass="0.01" x="0.013" y="0.023" z="0.023" material="blue"/>
+    <xacro:fixed_joint name="servo_adapter_to_servo" parent="servo_adapter" child="servo"
+                       origin_position="-0.011 0 0.012"/>
+    <xacro:mesh_link name="ultrasonic_adapter" package="robot_description" file="description/meshes/servo_to_ultrasonic_adapter.stl"
+                     origin_orientation="1.5708 0 -1.5708"/>
+    <xacro:fixed_joint name="servo_to_ultrasonic_adapter" parent="servo" child="ultrasonic_adapter"
+                       origin_position="0.005 0 0.035"/>
+    <xacro:box_link name="ultrasonic" mass="0.01" x="0.0015" y="0.045" z="0.020" material="blue"/>
+    <xacro:fixed_joint name="ultrasonic_adapter_to_ultrasonic" parent="ultrasonic_adapter" child="ultrasonic"
+                       origin_position="-0.005 0 0"/>
+    <xacro:box_link name="camera" mass="0.01" x="0.001" y="0.025" z="0.024" material="blue"
+                    origin_orientation="0 0 -0.1745"/> <!-- 10 deg -->
+    <xacro:fixed_joint name="camera_adapter_to_camera" child="camera" parent="camera_adapter"
+                       origin_position="-0.007 0 0.014"/>
+    <xacro:cylinder_link name="lidar" mass="0.01" radius="0.031" length="0.02" material="blue"/>
+    <xacro:fixed_joint name="lidar_to_lidar_adapter" child="lidar" parent="lidar_adapter"
+                       origin_position="0.010 0 0.040"/>
+    <!-- <xacro:box_link name="line_tracking_${suffix}" mass="0.001" x="0.01" y="0.01" z="0.01" material="black"/>
+    <xacro:fixed_joint name="line_tracking_${suffix}" child="line_tracking_${suffix}" origin_position="${origin}" origin_orientation="0 1.57 0"/> -->
 </xacro:macro>
 </robot>

File: src/robot_description/description/robot.xacro (robot description, xacro)
@@ -2,4 +2,5 @@
 <robot xmlns:xacro="http://www.ros.org/wiki/xacro" name="robot">
     <xacro:arg name="use_sim" default="false"/>
+    <!-- includes -->
     <xacro:include filename="properties.xacro"/>
     <xacro:include filename="component_macros.xacro"/>
@@ -7,9 +8,10 @@
     <xacro:include filename="ros2_control.xacro"/>
     <xacro:include filename="frame.xacro"/>
+    <xacro:include filename="gazebo.xacro"/>
     <!-- robot -->
     <xacro:coordinate_frames/>
-    <xacro:robot_chassis/>
-    <xacro:motors_and_wheels/>
-    <xacro:ros2_control_diffdrive/>
+    <xacro:robot_description/>
+    <xacro:ros2_control_diffdrive_plugin/>
+    <xacro:gazebo_plugins/>
     <!-- <xacro:box_link name="chassis" mass="2" x="${chassis_length}" y="${chassis_width}" z="${chassis_height}" material="black"/>   -->
     <!-- <xacro:imu/> -->
