Commit message: Update: xacro robot description is now caught up with new robot

File: src/robot_description/description/ros2_control.xacro (robot description, xacro)
@@ -1,38 +1,63 @@
 <?xml version="1.0"?>
 <robot xmlns:xacro="http://www.ros.org/wiki/xacro">
-  <xacro:macro name="ros2_control_diffdrive">
-    <ros2_control name="ros2_control_diffdrive" type="system">
-      <hardware>
-          <plugin>ros2_control_diffdrive_encoder_plugin/DiffDriveHardware</plugin>
-          <param name="motor_left_enable_pin">4</param>
-          <param name="motor_left_forward_pin">21</param>
-          <param name="motor_left_backward_pin">26</param>
-          <param name="motor_right_enable_pin">17</param>
-          <param name="motor_right_forward_pin">18</param>
-          <param name="motor_right_backward_pin">27</param>
-          <param name="motor_rpm">130</param>
-          <param name="encoder_left_green_pin">22</param>
-          <param name="encoder_left_yellow_pin">23</param>
-          <param name="encoder_right_green_pin">24</param>
-          <param name="encoder_right_yellow_pin">25</param>
-          <param name="encoder_tics_per_rotation">494</param>
-      </hardware>
-      <joint name="left_wheel_joint">
-          <command_interface name="velocity">
-              <param name="min">-100</param>
-              <param name="max">100</param>
-          </command_interface>
-          <state_interface name="position"/>
-          <state_interface name="velocity"/>
-      </joint>
-      <joint name="right_wheel_joint">
-          <command_interface name="velocity">
-              <param name="min">-100</param>
-              <param name="max">100</param>
-          </command_interface>
-          <state_interface name="position"/>
-          <state_interface name="velocity"/>
-      </joint>
-    </ros2_control>
+  <xacro:macro name="ros2_control_diffdrive_plugin">
+    <xacro:if value="$(arg use_sim)">
+        <ros2_control name="ros2_control_diffdrive" type="system">
+        <hardware>
+            <plugin>ros2_control_diffdrive_encoder_plugin/DiffDriveHardware</plugin>
+            <param name="motor_left_enable_pin">4</param>
+            <param name="motor_left_forward_pin">21</param>
+            <param name="motor_left_backward_pin">26</param>
+            <param name="motor_right_enable_pin">17</param>
+            <param name="motor_right_forward_pin">18</param>
+            <param name="motor_right_backward_pin">27</param>
+            <param name="motor_rpm">130</param>
+            <param name="encoder_left_green_pin">22</param>
+            <param name="encoder_left_yellow_pin">23</param>
+            <param name="encoder_right_green_pin">24</param>
+            <param name="encoder_right_yellow_pin">25</param>
+            <param name="encoder_tics_per_rotation">494</param>
+        </hardware>
+        <joint name="left_motor_bracket_to_left_wheel">
+            <command_interface name="velocity">
+                <param name="min">-100</param>
+                <param name="max">100</param>
+            </command_interface>
+            <state_interface name="position"/>
+            <state_interface name="velocity"/>
+        </joint>
+        <joint name="right_motor_bracket_to_right_wheel">
+            <command_interface name="velocity">
+                <param name="min">-100</param>
+                <param name="max">100</param>
+            </command_interface>
+            <state_interface name="position"/>
+            <state_interface name="velocity"/>
+        </joint>
+        </ros2_control>
+    </xacro:if>
+    <xacro:unless value="$(arg use_sim)">
+        <ros2_control name="ros2_control_diffdrive" type="system">
+            <hardware>
+                <plugin>gz_ros2_control/GazeboSimSystem</plugin>
+            </hardware>
+            <joint name="left_motor_bracket_to_left_wheel">
+                <command_interface name="velocity">
+                    <param name="min">-100</param>
+                    <param name="max">100</param>
+                </command_interface>
+                <state_interface name="position"/>
+                <state_interface name="velocity"/>
+            </joint>
+            <joint name="right_motor_bracket_to_right_wheel">
+                <command_interface name="velocity">
+                    <param name="min">-100</param>
+                    <param name="max">100</param>
+                </command_interface>
+                <state_interface name="position"/>
+                <state_interface name="velocity"/>
+            </joint>
+        </ros2_control>
+    </xacro:unless>
   </xacro:macro>
 </robot>

Commit message: Remove: unused stuff from robot description files Fix: small fixes in values, and polish

File: src/robot_description/description/component_macros.xacro (robot description, xacro)
@@ -77,10 +77,10 @@
 <xacro:macro name="mesh_link" params="name package file material:=red scale:=0.001 origin_position:='0 0 0' origin_orientation:='0 0 0'">
     <link name="${name}">
-        <!-- <inertial>
-            <mass value="${mass}" />
-            <inertia ixx="${(1/12) * mass * (y*y+z*z)}" ixy="0.0" ixz="0.0"
-                     iyy="${(1/12) * mass * (x*x+z*z)}" iyz="0.0"
-                     izz="${(1/12) * mass * (x*x+y*y)}" />
-        </inertial> -->
+        <inertial>
+            <mass value="10" />
+            <inertia ixx="0.0" ixy="0.0" ixz="0.0"
+                     iyy="0.0" iyz="0.0"
+                     izz="0.0" />
+        </inertial>
         <visual>
             <geometry>
@@ -113,113 +113,6 @@
     </joint>
 </xacro:macro>
-<xacro:macro name="floating_joint" params="name parent child origin_position:='0 0 0' origin_orientation:='0 0 0'">
-    <joint name="${name}" type="floating">
-        <parent link="${parent}"/>
-        <child link="${child}"/>
-        <origin xyz="${origin_position}" rpy="${origin_orientation}"/>
-    </joint>
-</xacro:macro>
-<!-- output components -->
-<xacro:macro name="diff_drive_old" params="">
-    <xacro:cylinder_link name="left_front_wheel" mass="0.05" radius="${wheel_radius}" length="0.02" material="yellow"/>
-    <xacro:continuous_joint name="left_front_wheel" child="left_front_wheel" origin_position="0.045 0.075 -0.025" origin_orientation="-1.5707 0 0" axis="0 0 1"/>
-    <xacro:cylinder_link name="right_front_wheel" mass="0.05" radius="${wheel_radius}" length="0.02" material="yellow"/>
-    <xacro:continuous_joint name="right_front_wheel" child="right_front_wheel" origin_position="0.045 -0.075 -0.025" origin_orientation="-1.5707 0 0" axis="0 0 1"/>
-    <xacro:cylinder_link name="left_rear_wheel" mass="0.05" radius="${wheel_radius}" length="0.02" material="yellow"/>
-    <xacro:continuous_joint name="left_rear_wheel" child="left_rear_wheel" origin_position="-0.05 0.075 -0.025" origin_orientation="-1.5707 0 0" axis="0 0 1"/>
-    <xacro:cylinder_link name="right_rear_wheel" mass="0.05" radius="${wheel_radius}" length="0.02" material="yellow"/>
-    <xacro:continuous_joint name="right_rear_wheel" child="right_rear_wheel" origin_position="-0.05 -0.075 -0.025" origin_orientation="-1.5707 0 0" axis="0 0 1"/>
-    <xacro:if value="$(arg use_sim)">
-        <ros2_control name="GazeboSimSystem" type="system">
-            <hardware>
-                <plugin>gz_ros2_control/GazeboSimSystem</plugin>
-            </hardware>
-            <joint name="left_front_wheel_joint">
-                <command_interface name="velocity">
-                    <param name="min">-100</param>
-                    <param name="max">100</param>
-                </command_interface>
-                <state_interface name="position"/>
-                <state_interface name="velocity"/>
-            </joint>
-            <joint name="right_front_wheel_joint">
-                <command_interface name="velocity">
-                    <param name="min">-100</param>
-                    <param name="max">100</param>
-                </command_interface>
-                <state_interface name="position"/>
-                <state_interface name="velocity"/>
-            </joint>
-            <joint name="left_rear_wheel_joint">
-                <command_interface name="velocity">
-                    <param name="min">-100</param>
-                    <param name="max">100</param>
-                </command_interface>
-                <state_interface name="position"/>
-                <state_interface name="velocity"/>
-            </joint>
-            <joint name="right_rear_wheel_joint">
-                <command_interface name="velocity">
-                    <param name="min">-100</param>
-                    <param name="max">100</param>
-                </command_interface>
-                <state_interface name="position"/>
-                <state_interface name="velocity"/>
-            </joint>
-        </ros2_control>
-    </xacro:if>
-    <xacro:unless value="$(arg use_sim)">
-        <ros2_control name="GazeboRealSystem" type="system">
-            <hardware>
-                <plugin>adeept_awr_diffdrive_control_plugin/AdeeptDiffDriveHardware</plugin>
-                <param name="motor_left_enable_pin">4</param>
-                <param name="motor_left_forward_pin">21</param>
-                <param name="motor_left_backward_pin">26</param>
-                <param name="motor_right_enable_pin">17</param>
-                <param name="motor_right_forward_pin">18</param>
-                <param name="motor_right_backward_pin">27</param>
-                <param name="max_motor_rotation_speed">18.0</param>
-            </hardware>
-            <joint name="left_front_wheel_joint">
-                <command_interface name="velocity">
-                    <param name="min">-100</param>
-                    <param name="max">100</param>
-                </command_interface>
-            </joint>
-            <joint name="right_front_wheel_joint">
-                <command_interface name="velocity">
-                    <param name="min">-100</param>
-                    <param name="max">100</param>
-                </command_interface>
-            </joint>
-            <joint name="left_rear_wheel_joint">
-                <command_interface name="velocity">
-                    <param name="min">-100</param>
-                    <param name="max">100</param>
-                </command_interface>
-                </joint>
-            <joint name="right_rear_wheel_joint">
-                <command_interface name="velocity">
-                    <param name="min">-100</param>
-                    <param name="max">100</param>
-                </command_interface>
-            </joint>
-        </ros2_control>
-    </xacro:unless>
-    <gazebo>
-        <plugin filename="/opt/ros/jazzy/lib/libgz_ros2_control-system.so" name="gz_ros2_control::GazeboSimROS2ControlPlugin">
-            <parameters>$(find adeept_awr_diffdrive_control_plugin)/config/controllers.yaml</parameters>
-            <parameters>$(find adeept_awr_diffdrive_control_plugin)/config/controllers_sim.yaml</parameters>
-            <ros>
-                <remapping>/diff_drive_controller/cmd_vel:=/cmd_vel</remapping>
-                <!-- <remapping>/robot_description:=/controller_manager/robot_description</remapping> no longer needed -->
-            </ros>
-        </plugin>
-    </gazebo>
-</xacro:macro>
-<xacro:macro name="servo" params="name parent:=chassis child
-                                origin_position:='0 0 0' origin_orientation:='0 0 0' axis='0 0 0'
-                                limit_lower:=-3.14, limit_upper:=3.14">
-    <joint name="${name}_joint" type="revolute">
+<xacro:macro name="revolute_joint" params="name parent child origin_position:='0 0 0' origin_orientation:='0 0 0' axis='0 0 0' limit_lower:=-3.14, limit_upper:=3.14">
+    <joint name="${name}" type="revolute">
         <parent link="${parent}"/>
         <child link="${child}"/>
@@ -228,9 +121,4 @@
         <limit lower="${limit_lower}" upper="${limit_upper}" effort="10" velocity="3.14"/>
     </joint>
-    <gazebo>
-        <plugin name="ignition::gazebo::systems::JointController" filename="libignition-gazebo-joint-controller-system.so">
-            <joint_name>${name}_joint</joint_name>
-        </plugin>
-    </gazebo>
 </xacro:macro>
 </robot>

File: src/robot_description/description/frame.xacro (robot description, xacro)
@@ -67,5 +67,5 @@
                        origin_position="0.0085 -0.040 0.1075"/>
 </xacro:macro>
-<!-- battery model (mainly included weight and visual) -->
+<!-- battery model (mainly included for weight and visual) -->
 <xacro:macro name="power_source">
     <xacro:mesh_link name="battery_base" package="robot_description" file="description/meshes/orp_battery_base.stl"
@@ -86,5 +86,5 @@
                        origin_position="0 0 -0.053"/>
 </xacro:macro>
-<!-- wheels are important here they are used by ros2_control, motors are just visual -->
+<!-- most important part here are the wheels since they are used by ros2_control, motors are just visual -->
 <xacro:macro name="motors_and_wheels">
     <xacro:cylinder_link name="left_motor" mass="20" radius="0.010" length="0.050"
@@ -92,5 +92,5 @@
     <xacro:fixed_joint name="left_motor_bracket_to_left_motor" parent="left_motor_bracket" child="left_motor"
                        origin_position="0 -0.025 -0.0175"/>
-    <xacro:cylinder_link name="left_wheel" mass="20" radius="0.025" length="0.020"
+    <xacro:cylinder_link name="left_wheel" mass="20" radius="0.0345" length="0.020"
                          origin_orientation="1.5708 0 0"/>
     <xacro:continuous_joint name="left_motor_bracket_to_left_wheel" parent="left_motor_bracket" child="left_wheel"
@@ -100,12 +100,12 @@
     <xacro:fixed_joint name="right_motor_bracket_to_right_motor" parent="right_motor_bracket" child="right_motor"
                        origin_position="0 0.025 -0.0175"/>
-    <xacro:cylinder_link name="right_wheel" mass="20" radius="0.025" length="0.020"
+    <xacro:cylinder_link name="right_wheel" mass="20" radius="0.0345" length="0.020"
                          origin_orientation="1.5708 0 0"/>
     <xacro:continuous_joint name="right_motor_bracket_to_right_wheel" parent="right_motor_bracket" child="right_wheel"
                             origin_position="0 -0.025 -0.0175" axis="0 1 0"/>
-    <xacro:ball_link name="front_caster_wheel" mass="1" radius="0.010"/>
+    <xacro:ball_link name="front_caster_wheel" mass="1" radius="0.015"/>
     <xacro:fixed_joint name="front_caster_adapter_to_front_caster_wheel" parent="front_caster_adapter" child="front_caster_wheel"
                        origin_position="0 0 -0.035"/>
-    <xacro:ball_link name="back_caster_wheel" mass="1" radius="0.010"/>
+    <xacro:ball_link name="back_caster_wheel" mass="1" radius="0.015"/>
     <xacro:fixed_joint name="back_caster_adapter_to_back_caster_wheel" parent="back_caster_adapter" child="back_caster_wheel"
                        origin_position="0 0 -0.035"/>
@@ -118,6 +118,6 @@
     <xacro:mesh_link name="ultrasonic_adapter" package="robot_description" file="description/meshes/servo_to_ultrasonic_adapter.stl"
                      origin_orientation="1.5708 0 -1.5708"/>
-    <xacro:fixed_joint name="servo_to_ultrasonic_adapter" parent="servo" child="ultrasonic_adapter"
-                       origin_position="0.005 0 0.035"/>
+    <xacro:revolute_joint name="servo_to_ultrasonic_adapter" parent="servo" child="ultrasonic_adapter"
+                          origin_position="0.005 0 0.035" axis="0 0 1" limit_lower="-3.14" limit_upper="3.14"/>
     <xacro:box_link name="ultrasonic" mass="0.01" x="0.0015" y="0.045" z="0.020" material="blue"/>
     <xacro:fixed_joint name="ultrasonic_adapter_to_ultrasonic" parent="ultrasonic_adapter" child="ultrasonic"

File: src/robot_description/description/gazebo.xacro (robot description, xacro)
@@ -2,14 +2,17 @@
 <robot xmlns:xacro="http://www.ros.org/wiki/xacro">
     <xacro:macro name="gazebo_plugins">
-    <gazebo>
-        <plugin filename="/opt/ros/jazzy/lib/libgz_ros2_control-system.so" name="gz_ros2_control::GazeboSimROS2ControlPlugin">
-            <parameters>$(find ros2_control_diffdrive_encoder_plugin)/bringup/config/controllers.yaml</parameters>
-            <parameters>$(find ros2_control_diffdrive_encoder_plugin)/bringup/config/controllers_sim.yaml</parameters>
-            <ros>
-                <remapping>/diff_drive_controller/cmd_vel:=/cmd_vel</remapping>
-                <!-- <remapping>/robot_description:=/controller_manager/robot_description</remapping> no longer needed -->
-            </ros>
-        </plugin>
-    </gazebo>
+    <xacro:if value="$(arg use_sim)">
+        <gazebo>
+            <plugin filename="/opt/ros/jazzy/lib/libgz_ros2_control-system.so" name="gz_ros2_control::GazeboSimROS2ControlPlugin">
+                <parameters>$(find ros2_control_diffdrive_encoder_plugin)/bringup/config/controllers.yaml</parameters>
+                <parameters>$(find ros2_control_diffdrive_encoder_plugin)/bringup/config/controllers_sim.yaml</parameters>
+                <ros>
+                    <remapping>/diff_drive_controller/cmd_vel:=/cmd_vel</remapping>
+                    <!-- <remapping>/diff_drive_controller/odom:=/odom</remapping> -->
+                    <!-- <remapping>/robot_description:=/controller_manager/robot_description</remapping> no longer needed -->
+                </ros>
+            </plugin>
+        </gazebo>
+    </xacro:if>
     <gazebo reference="lidar">
         <sensor name='gpu_lidar' type='gpu_lidar'>
@@ -44,4 +47,9 @@
             </lidar>
         </sensor>
+    </gazebo>
+    <gazebo>
+        <plugin name="ignition::gazebo::systems::JointController" filename="libignition-gazebo-joint-controller-system.so">
+            <joint_name>servo_to_ultrasonic_adapter</joint_name>
+        </plugin>
     </gazebo>
     <gazebo reference="ultrasonic">
@@ -78,5 +86,5 @@
         </sensor>
     </gazebo>
-<gazebo reference="camera">
+    <gazebo reference="camera">
         <sensor name='camera' type='camera'>
             <topic>simulator_camera</topic>

File: src/robot_description/description/properties.xacro (robot description, xacro)
@@ -1,11 +1,11 @@
 <?xml version="1.0"?>
 <robot xmlns:xacro="http://ros.org/wiki/xacro">
-    <xacro:property name="chassis_length" value="0.13" />
-    <xacro:property name="chassis_width" value="0.12" />
-    <xacro:property name="chassis_height" value="0.075" />
-    <xacro:property name="wheel_separation" value="0.15" />
-    <xacro:property name="wheel_radius" value="0.035" />
+    <xacro:property name="wheel_separation" value="0.213" />
+    <xacro:property name="wheel_radius" value="0.069" />
     <material name="red">
         <color rgba="1.0 0.0 0.0 1.0"/>
+    </material>
+    <material name="green">
+        <color rgba="0.0 1.0 0.0 1.0"/>
     </material>
     <material name="blue">
@@ -15,6 +15,6 @@
         <color rgba="0.01 0.01 0.01 1.0"/>
     </material>
-    <material name="yellow">
-        <color rgba="1.0 1.0 0.0 1.0"/>
+    <material name="white">
+        <color rgba="1.0 1.0 1.0 1.0"/>
     </material>
 </robot>

File: src/robot_description/description/robot.xacro (robot description, xacro)
@@ -5,7 +5,6 @@
     <xacro:include filename="properties.xacro"/>
     <xacro:include filename="component_macros.xacro"/>
-    <xacro:include filename="sensors_and_acuators.xacro"/>
+    <xacro:include filename="frame.xacro"/>
     <xacro:include filename="ros2_control.xacro"/>
-    <xacro:include filename="frame.xacro"/>
     <xacro:include filename="gazebo.xacro"/>
     <!-- robot -->
@@ -14,6 +13,3 @@
     <xacro:ros2_control_diffdrive_plugin/>
     <xacro:gazebo_plugins/>
-    <!-- <xacro:box_link name="chassis" mass="2" x="${chassis_length}" y="${chassis_width}" z="${chassis_height}" material="black"/>   -->
-    <!-- <xacro:imu/> -->
-    <!-- <xacro:fixed_joint name="chassis" parent="base_link" child="chassis" origin_position="0 0 0.1"/> -->
 </robot>

File: src/robot_description/description/ros2_control.xacro (robot description, xacro)
@@ -1,6 +1,31 @@
 <?xml version="1.0"?>
 <robot xmlns:xacro="http://www.ros.org/wiki/xacro">
-  <xacro:macro name="ros2_control_diffdrive_plugin">
+<xacro:macro name="ros2_control_diffdrive_plugin">
+    <!-- simulation plugin -->
     <xacro:if value="$(arg use_sim)">
+        <ros2_control name="ros2_control_diffdrive" type="system">
+            <hardware>
+                <plugin>gz_ros2_control/GazeboSimSystem</plugin>
+            </hardware>
+            <joint name="left_motor_bracket_to_left_wheel">
+                <command_interface name="velocity">
+                    <param name="min">-100</param>
+                    <param name="max">100</param>
+                </command_interface>
+                <state_interface name="position"/>
+                <state_interface name="velocity"/>
+            </joint>
+            <joint name="right_motor_bracket_to_right_wheel">
+                <command_interface name="velocity">
+                    <param name="min">-100</param>
+                    <param name="max">100</param>
+                </command_interface>
+                <state_interface name="position"/>
+                <state_interface name="velocity"/>
+            </joint>
+        </ros2_control>
+    </xacro:if>
+    <!-- real robot plugin -->
+    <xacro:unless value="$(arg use_sim)">
         <ros2_control name="ros2_control_diffdrive" type="system">
         <hardware>
@@ -36,28 +61,5 @@
         </joint>
         </ros2_control>
-    </xacro:if>
-    <xacro:unless value="$(arg use_sim)">
-        <ros2_control name="ros2_control_diffdrive" type="system">
-            <hardware>
-                <plugin>gz_ros2_control/GazeboSimSystem</plugin>
-            </hardware>
-            <joint name="left_motor_bracket_to_left_wheel">
-                <command_interface name="velocity">
-                    <param name="min">-100</param>
-                    <param name="max">100</param>
-                </command_interface>
-                <state_interface name="position"/>
-                <state_interface name="velocity"/>
-            </joint>
-            <joint name="right_motor_bracket_to_right_wheel">
-                <command_interface name="velocity">
-                    <param name="min">-100</param>
-                    <param name="max">100</param>
-                </command_interface>
-                <state_interface name="position"/>
-                <state_interface name="velocity"/>
-            </joint>
-        </ros2_control>
     </xacro:unless>
-  </xacro:macro>
+</xacro:macro>
 </robot>
