Commit message: Fix: many small, mostly naming changes and fixes Update: xacro ros2 control plugin to work with updated version  motor library Remove: remains of old servo controllers (both real using pyhton node and adafruit library, and simulator using gazebo plugin)

File: src/waferbot/waferbot_description/description/gazebo_plugins.xacro (robot description, xacro)
@@ -5,6 +5,5 @@
         <gazebo>
             <plugin filename="/opt/ros/jazzy/lib/libgz_ros2_control-system.so" name="gz_ros2_control::GazeboSimROS2ControlPlugin">
-                <parameters>$(find jga25_371_hardware_interface)/bringup/config/controllers.yaml</parameters>
-                <parameters>$(find jga25_371_hardware_interface)/bringup/config/controllers_sim.yaml</parameters>
+                <parameters>$(find waferbot_gazebo)/config/ros2_control_config.yaml</parameters>
                 <ros>
                     <remapping>/diff_drive_controller/cmd_vel:=/cmd_vel</remapping>

File: src/waferbot/waferbot_description/description/physical_components.xacro (robot description, xacro)
@@ -72,5 +72,5 @@
     <xacro:fixed_joint name="bottom_baseplate_to_top_baseplate" parent="bottom_baseplate" child="top_baseplate"
                        origin_position="0 0 0.105"/>
-    <xacro:mesh_link name="lidar_adapter" package="waferbot_description" file="description/meshes/orp_lidar.stl"
+    <xacro:mesh_link name="lidar_adapter" package="waferbot_description" file="description/meshes/orp_lidar_adapter.stl"
                      origin_orientation="1.5708 0 3.1415"/>
     <xacro:fixed_joint name="top_baseplate_to_lidar_adapter" parent="top_baseplate" child="lidar_adapter"

File: src/waferbot/waferbot_description/description/ros2_control_plugins.xacro (robot description, xacro)
@@ -9,16 +9,10 @@
             </hardware>
             <joint name="left_motor_bracket_to_left_wheel">
-                <command_interface name="velocity">
-                    <param name="min">-100</param>
-                    <param name="max">100</param>
-                </command_interface>
+                <command_interface name="velocity"/>
                 <state_interface name="position"/>
                 <state_interface name="velocity"/>
             </joint>
             <joint name="right_motor_bracket_to_right_wheel">
-                <command_interface name="velocity">
-                    <param name="min">-100</param>
-                    <param name="max">100</param>
-                </command_interface>
+                <command_interface name="velocity"/>
                 <state_interface name="position"/>
                 <state_interface name="velocity"/>
@@ -29,38 +23,35 @@
     <xacro:unless value="$(arg use_sim)">
         <ros2_control name="ros2_control_diffdrive" type="system">
-        <hardware>
-            <plugin>jga25_371_hardware_interface/DiffDriveHardware</plugin>
-            <param name="motor_left_enable_pin">17</param>
-            <param name="motor_left_forward_pin">27</param>
-            <param name="motor_left_backward_pin">18</param>
-            <param name="motor_right_enable_pin">4</param>
-            <param name="motor_right_forward_pin">26</param>
-            <param name="motor_right_backward_pin">21</param>
-            <param name="motor_rpm">130</param>
-            <param name="encoder_left_green_pin">25</param>
-            <param name="encoder_left_yellow_pin">24</param>
-            <param name="encoder_right_green_pin">22</param>
-            <param name="encoder_right_yellow_pin">23</param>
-            <param name="encoder_tics_per_rotation">1976</param>
-        </hardware>
-        <joint name="left_motor_bracket_to_left_wheel">
-            <command_interface name="velocity">
-                <param name="min">-100</param>
-                <param name="max">100</param>
-            </command_interface>
-            <state_interface name="position"/>
-            <state_interface name="velocity"/>
-        </joint>
-        <joint name="right_motor_bracket_to_right_wheel">
-            <command_interface name="velocity">
-                <param name="min">-100</param>
-                <param name="max">100</param>
-            </command_interface>
-            <state_interface name="position"/>
-            <state_interface name="velocity"/>
-        </joint>
+            <hardware>
+                <plugin>jga25_371_hardware_interface/DiffDriveHardware</plugin>
+            </hardware>
+            <joint name="left_motor_bracket_to_left_wheel">
+                <command_interface name="velocity"/>
+                <state_interface name="position"/>
+                <state_interface name="velocity"/>
+                <param name="enable_pin">17</param>
+                <param name="forward_pin">27</param>
+                <param name="backward_pin">18</param>
+                <param name="encoder_A_pin">24</param>
+                <param name="encoder_B_pin">25</param>
+                <param name="motor_rpm">130</param>
+                <param name="encoder_tics_per_rotation">1976</param>
+            </joint>
+            <joint name="right_motor_bracket_to_right_wheel">
+                <command_interface name="velocity"/>
+                <state_interface name="position"/>
+                <state_interface name="velocity"/>
+                <param name="enable_pin">4</param>
+                <param name="forward_pin">26</param>
+                <param name="backward_pin">21</param>
+                <param name="encoder_A_pin">23</param>
+                <param name="encoder_B_pin">22</param>
+                <param name="motor_rpm">130</param>
+                <param name="encoder_tics_per_rotation">1976</param>
+            </joint>
         </ros2_control>
     </xacro:unless>
 </xacro:macro>
+<!-- todo: this need to be done for simulator -->
 <xacro:macro name="ros2_control_pca9685">
     <ros2_control name="ros2_control_pca9685" type="system">
