Commit message: Fix: small fixes, diff_drive_controller had slightly wrong wheel separation and radius params orgre sensor system should be declared once per world, having that in xacro leads to crash when spawning second robot

File: src/waferbot/waferbot_description/xacro/gazebo_plugins.xacro (robot description, xacro)
@@ -12,9 +12,4 @@
         </gazebo>
     </xacro:if>
-    <gazebo>
-        <plugin name='gz::sim::systems::Sensors' filename='ignition-gazebo-sensors-system'>
-            <render_engine>ogre2</render_engine>
-        </plugin>
-    </gazebo>
     <gazebo reference="imu">
         <sensor name="imu" type="imu">

File: src/waferbot/waferbot_description/xacro/properties.xacro (robot description, xacro)
@@ -1,6 +1,4 @@
 <?xml version="1.0"?>
 <robot xmlns:xacro="http://ros.org/wiki/xacro">
-    <xacro:property name="wheel_separation" value="0.213" />
-    <xacro:property name="wheel_radius" value="0.069" />
     <material name="red">
         <color rgba="1.0 0.0 0.0 1.0"/>
