Commit message: Update: models optimization new argument for xacro robot description, disables collision for all objects (most importantly mesh links, where mesh collision has huge performance impact), well most objects, of course there are exceptions for wheels, that overwrite this global parameter because wheels without collision are useless, this argument also disables camera plugin because it has big performance impact and is not required for multi robot orchestration

File: src/waferbot/waferbot_description/xacro/component_macros.xacro (robot description, xacro)
@@ -2,5 +2,5 @@
 <robot xmlns:xacro="http://ros.org/wiki/xacro">
 <!-- basic building blocks -->
-<xacro:macro name="box_link" params="name mass x y z material:=red origin_position:='0 0 0' origin_orientation:='0 0 0'">
+<xacro:macro name="box_link" params="name mass x y z material:=red origin_position:='0 0 0' origin_orientation:='0 0 0' use_collision:=${not $(arg optimize_sim_perf)}">
     <link name="${name}">
         <inertial>
@@ -18,13 +18,15 @@
             <origin xyz="${origin_position}" rpy="${origin_orientation}"/>
         </visual>
-        <collision>
-            <geometry>
-                <box size="${x} ${y} ${z}"/>
-            </geometry>
-            <origin xyz="${origin_position}" rpy="${origin_orientation}"/>
-        </collision>
+        <xacro:if value="${use_collision}">
+            <collision>
+                <geometry>
+                    <box size="${x} ${y} ${z}"/>
+                </geometry>
+                <origin xyz="${origin_position}" rpy="${origin_orientation}"/>
+            </collision>
+        </xacro:if>
     </link>
 </xacro:macro>
-<xacro:macro name="cylinder_link" params="name mass radius length material:=red origin_position:='0 0 0' origin_orientation:='0 0 0'">
+<xacro:macro name="cylinder_link" params="name mass radius length material:=red origin_position:='0 0 0' origin_orientation:='0 0 0' use_collision:=${not $(arg optimize_sim_perf)}">
     <link name="${name}">
         <inertial>
@@ -42,13 +44,15 @@
             <origin xyz="${origin_position}" rpy="${origin_orientation}"/>
         </visual>
-        <collision>
-            <geometry>
-                <cylinder radius="${radius}" length="${length}"/>
-            </geometry>
-            <origin xyz="${origin_position}" rpy="${origin_orientation}"/>
-        </collision>
+        <xacro:if value="${use_collision}">
+            <collision>
+                <geometry>
+                    <cylinder radius="${radius}" length="${length}"/>
+                </geometry>
+                <origin xyz="${origin_position}" rpy="${origin_orientation}"/>
+            </collision>
+        </xacro:if>
     </link>
 </xacro:macro>
-<xacro:macro name="ball_link" params="name mass radius material:=red origin_position:='0 0 0' origin_orientation:='0 0 0'">
+<xacro:macro name="ball_link" params="name mass radius material:=red origin_position:='0 0 0' origin_orientation:='0 0 0' use_collision:=${not $(arg optimize_sim_perf)}">
     <link name="${name}">
         <inertial>
@@ -67,13 +71,15 @@
             <origin xyz="${origin_position}" rpy="${origin_orientation}"/>
         </visual>
-        <collision>
-            <geometry>
-                <sphere radius="${radius}"/>
-            </geometry>
-            <origin xyz="${origin_position}" rpy="${origin_orientation}"/>
-        </collision>
+        <xacro:if value="${use_collision}">
+            <collision>
+                <geometry>
+                    <sphere radius="${radius}"/>
+                </geometry>
+                <origin xyz="${origin_position}" rpy="${origin_orientation}"/>
+            </collision>
+        </xacro:if>
     </link>
 </xacro:macro>
-<xacro:macro name="mesh_link" params="name package file material:=red scale:=0.001 origin_position:='0 0 0' origin_orientation:='0 0 0' mass:=0.020">
+<xacro:macro name="mesh_link" params="name package file material:=red scale:=0.001 origin_position:='0 0 0' origin_orientation:='0 0 0' mass:=0.020 use_collision:=${not $(arg optimize_sim_perf)}">
     <link name="${name}">
         <inertial>
@@ -90,10 +96,12 @@
             <origin xyz="${origin_position}" rpy="${origin_orientation}"/>
         </visual>
-        <collision>
-            <geometry>
-                <mesh filename="file://$(find ${package})/${file}" scale="${scale} ${scale} ${scale}"/>
-            </geometry>
-            <origin xyz="${origin_position}" rpy="${origin_orientation}"/>
-        </collision>
+        <xacro:if value="${use_collision}">
+            <collision>
+                <geometry>
+                    <mesh filename="file://$(find ${package})/${file}" scale="${scale} ${scale} ${scale}"/>
+                </geometry>
+                <origin xyz="${origin_position}" rpy="${origin_orientation}"/>
+            </collision>
+        </xacro:if>
     </link>
 </xacro:macro>

File: src/waferbot/waferbot_description/xacro/gazebo_plugins.xacro (robot description, xacro)
@@ -88,30 +88,32 @@
         </sensor>
     </gazebo>
-    <gazebo reference="camera">
-        <sensor name="camera_sensor" type="camera">
-            <update_rate>20</update_rate>
-            <topic>$(arg robot_name)/camera/image</topic>
-            <gz_frame_id>$(arg robot_name)/camera</gz_frame_id>
-            <camera>
-                <horizontal_fov>0.9328</horizontal_fov>
-                <image>
-                    <width>640</width>
-                    <height>480</height>
-                    <format>RGB_INT8</format>
-                </image>
-                <clip>
-                    <near>0.01</near>
-                    <far>100</far>
-                </clip>
-                <visibility_mask>4294967295</visibility_mask>
-                <lens>
-                    <type>stereographic</type>
-                    <scale_to_hfov>true</scale_to_hfov>
-                    <cutoff_angle>1.5708</cutoff_angle>
-                    <env_texture_size>256</env_texture_size>
-                </lens>
-            </camera>
-        </sensor>
-    </gazebo>
+    <xacro:unless value="$(arg optimize_sim_perf)">
+        <gazebo reference="camera">
+            <sensor name="camera_sensor" type="camera">
+                <update_rate>20</update_rate>
+                <topic>$(arg robot_name)/camera/image</topic>
+                <gz_frame_id>$(arg robot_name)/camera</gz_frame_id>
+                <camera>
+                    <horizontal_fov>0.9328</horizontal_fov>
+                    <image>
+                        <width>640</width>
+                        <height>480</height>
+                        <format>RGB_INT8</format>
+                    </image>
+                    <clip>
+                        <near>0.01</near>
+                        <far>100</far>
+                    </clip>
+                    <visibility_mask>4294967295</visibility_mask>
+                    <lens>
+                        <type>stereographic</type>
+                        <scale_to_hfov>true</scale_to_hfov>
+                        <cutoff_angle>1.5708</cutoff_angle>
+                        <env_texture_size>256</env_texture_size>
+                    </lens>
+                </camera>
+            </sensor>
+        </gazebo>
+    </xacro:unless>
 </xacro:macro>
 </robot>

File: src/waferbot/waferbot_description/xacro/physical_components.xacro (robot description, xacro)
@@ -3,4 +3,18 @@
 <!-- orp baseplates and adapters, all with fixed joints -->
 <xacro:macro name="chassis">
+    <xacro:if value="$(arg optimize_sim_perf)">
+        <link name="box_collision_approximation">
+            <collision>
+                <geometry>
+                    <box size="0.215 0.185 0.1125"/>
+                </geometry>
+            </collision>
+        </link>
+        <joint name="base_link_to_box_collision_approximation" type="fixed">
+            <parent link="base_link"/>
+            <child link="box_collision_approximation"/>
+            <origin xyz="0 0 0.05625" rpy="0 0 0"/>
+        </joint>
+    </xacro:if>
     <xacro:mesh_link name="bottom_baseplate" package="waferbot_description" file="meshes/orp_baseplate.stl"
                      mass="0.095" origin_orientation="1.5708 0 1.5708"/>
@@ -81,15 +95,15 @@
 <xacro:macro name="accurators">
     <xacro:cylinder_link name="left_wheel" mass="0.035" radius="0.0325" length="0.026"
-                         origin_orientation="1.5708 0 0"/>
+                         origin_orientation="1.5708 0 0" use_collision="true"/>
     <xacro:continuous_joint name="left_motor_bracket_to_left_wheel" parent="left_motor_bracket" child="left_wheel"
                             origin_position="0.020 0.023 -0.020" axis="0 1 0"/>
     <xacro:cylinder_link name="right_wheel" mass="0.035" radius="0.0325" length="0.026"
-                         origin_orientation="1.5708 0 0"/>
+                         origin_orientation="1.5708 0 0" use_collision="true"/>
     <xacro:continuous_joint name="right_motor_bracket_to_right_wheel" parent="right_motor_bracket" child="right_wheel"
                             origin_position="-0.020 -0.023 -0.020" axis="0 1 0"/>
-    <xacro:ball_link name="front_caster_wheel" mass="0.010" radius="0.015"/>
+    <xacro:ball_link name="front_caster_wheel" mass="0.010" radius="0.015" use_collision="true"/>
     <xacro:fixed_joint name="front_caster_adapter_to_front_caster_wheel" parent="front_caster_adapter" child="front_caster_wheel"
                        origin_position="0 0 -0.035"/>
-    <xacro:ball_link name="back_caster_wheel" mass="0.010" radius="0.015"/>
+    <xacro:ball_link name="back_caster_wheel" mass="0.010" radius="0.015" use_collision="true"/>
     <xacro:fixed_joint name="back_caster_adapter_to_back_caster_wheel" parent="back_caster_adapter" child="back_caster_wheel"
                        origin_position="0 0 -0.035"/>

File: src/waferbot/waferbot_description/xacro/waferbot.xacro (robot description, xacro)
@@ -1,6 +1,7 @@
 <?xml version="1.0"?>
 <robot xmlns:xacro="http://www.ros.org/wiki/xacro" name="$(arg robot_name)">
-    <xacro:arg name="use_sim" default="false"/>
     <xacro:arg name="robot_name" default="waferbot"/>
+    <xacro:arg name="use_sim" default="False"/>
+    <xacro:arg name="optimize_sim_perf" default="False"/>
     <!-- includes -->
     <xacro:include filename="properties.xacro"/>

Commit message: Fixes fix: motion executor config accuracy reduced to account for slower system fix: image_compressor converts rgb to brg so the colors are not switched fix: rmf robot adapter now publishes navigate_to_pose including yaw parameter fix: wheel odometry drift in simulator still not good enough, only viable fix is hacky, increasing weight of wheels to 10kg, commit also adds stuff like friction but that does not seem to do much difference update: navigation config split into two, because having one does not seem to be possible update: multi_robot_rviz config now in final version, with all six robots, map costmap, pre robot local scan model update: ultrasonic interpreter helper node for gazebo updated to not publish inf and to carry over header from gazebo scan source

File: src/waferbot/waferbot_description/xacro/component_macros.xacro (robot description, xacro)
@@ -2,5 +2,5 @@
 <robot xmlns:xacro="http://ros.org/wiki/xacro">
 <!-- basic building blocks -->
-<xacro:macro name="box_link" params="name mass x y z material:=red origin_position:='0 0 0' origin_orientation:='0 0 0' use_collision:=${not $(arg optimize_sim_perf)}">
+<xacro:macro name="box_link" params="name mass x y z material:=red origin_position:='0 0 0' origin_orientation:='0 0 0' use_collision:=${not $(arg optimize_sim_perf)} friction:='1.0'">
     <link name="${name}">
         <inertial>
@@ -23,4 +23,12 @@
                     <box size="${x} ${y} ${z}"/>
                 </geometry>
+                <surface>
+                    <friction>
+                        <ode>
+                            <mu>${friction}</mu>
+                            <mu2>${friction}</mu2>
+                        </ode>
+                    </friction>
+                </surface>
                 <origin xyz="${origin_position}" rpy="${origin_orientation}"/>
             </collision>
@@ -28,5 +36,5 @@
     </link>
 </xacro:macro>
-<xacro:macro name="cylinder_link" params="name mass radius length material:=red origin_position:='0 0 0' origin_orientation:='0 0 0' use_collision:=${not $(arg optimize_sim_perf)}">
+<xacro:macro name="cylinder_link" params="name mass radius length material:=red origin_position:='0 0 0' origin_orientation:='0 0 0' use_collision:=${not $(arg optimize_sim_perf)} friction:='1.0'">
     <link name="${name}">
         <inertial>
@@ -49,4 +57,12 @@
                     <cylinder radius="${radius}" length="${length}"/>
                 </geometry>
+                <surface>
+                    <friction>
+                        <ode>
+                            <mu>${friction}</mu>
+                            <mu2>${friction}</mu2>
+                        </ode>
+                    </friction>
+                </surface>
                 <origin xyz="${origin_position}" rpy="${origin_orientation}"/>
             </collision>
@@ -54,5 +70,5 @@
     </link>
 </xacro:macro>
-<xacro:macro name="ball_link" params="name mass radius material:=red origin_position:='0 0 0' origin_orientation:='0 0 0' use_collision:=${not $(arg optimize_sim_perf)}">
+<xacro:macro name="ball_link" params="name mass radius material:=red origin_position:='0 0 0' origin_orientation:='0 0 0' use_collision:=${not $(arg optimize_sim_perf)} friction:='1.0'">
     <link name="${name}">
         <inertial>
@@ -76,4 +92,12 @@
                     <sphere radius="${radius}"/>
                 </geometry>
+                <surface>
+                    <friction>
+                        <ode>
+                            <mu>${friction}</mu>
+                            <mu2>${friction}</mu2>
+                        </ode>
+                    </friction>
+                </surface>
                 <origin xyz="${origin_position}" rpy="${origin_orientation}"/>
             </collision>
@@ -81,11 +105,11 @@
     </link>
 </xacro:macro>
-<xacro:macro name="mesh_link" params="name package file material:=red scale:=0.001 origin_position:='0 0 0' origin_orientation:='0 0 0' mass:=0.020 use_collision:=${not $(arg optimize_sim_perf)}">
+<xacro:macro name="mesh_link" params="name package file material:=red scale:=0.001 origin_position:='0 0 0' origin_orientation:='0 0 0' mass:=0.020 use_collision:=${not $(arg optimize_sim_perf)} friction:='1.0'">
     <link name="${name}">
         <inertial>
             <mass value="${mass}" />
-            <inertia ixx="0.0" ixy="0.0" ixz="0.0"
-                     iyy="0.0" iyz="0.0"
-                     izz="0.0" />
+            <inertia ixx="${(1/12) * mass}" ixy="0.0" ixz="0.0"
+                     iyy="${(1/12) * mass}" iyz="0.0"
+                     izz="${(1/12) * mass}" />
         </inertial>
         <visual>
@@ -101,4 +125,12 @@
                     <mesh filename="file://$(find ${package})/${file}" scale="${scale} ${scale} ${scale}"/>
                 </geometry>
+                <surface>
+                    <friction>
+                        <ode>
+                            <mu>${friction}</mu>
+                            <mu2>${friction}</mu2>
+                        </ode>
+                    </friction>
+                </surface>
                 <origin xyz="${origin_position}" rpy="${origin_orientation}"/>
             </collision>

File: src/waferbot/waferbot_description/xacro/physical_components.xacro (robot description, xacro)
@@ -94,16 +94,17 @@
 <!-- continuous or revolut joints, ros2_control uses these -->
 <xacro:macro name="accurators">
-    <xacro:cylinder_link name="left_wheel" mass="0.035" radius="0.0325" length="0.026"
+    <!-- mass hack on wheels, fixes odom drift, seems ode (gazebo physics engine) is not a fan of having two casters on one robot -->
+    <xacro:cylinder_link name="left_wheel" mass="10.035" radius="0.0325" length="0.026" friction="5.0"
                          origin_orientation="1.5708 0 0" use_collision="true"/>
     <xacro:continuous_joint name="left_motor_bracket_to_left_wheel" parent="left_motor_bracket" child="left_wheel"
                             origin_position="0.020 0.023 -0.020" axis="0 1 0"/>
-    <xacro:cylinder_link name="right_wheel" mass="0.035" radius="0.0325" length="0.026"
+    <xacro:cylinder_link name="right_wheel" mass="10.035" radius="0.0325" length="0.026" friction="5.0"
                          origin_orientation="1.5708 0 0" use_collision="true"/>
     <xacro:continuous_joint name="right_motor_bracket_to_right_wheel" parent="right_motor_bracket" child="right_wheel"
                             origin_position="-0.020 -0.023 -0.020" axis="0 1 0"/>
-    <xacro:ball_link name="front_caster_wheel" mass="0.010" radius="0.015" use_collision="true"/>
+    <xacro:ball_link name="front_caster_wheel" mass="0.010" radius="0.015" friction="0.01" use_collision="true"/>
     <xacro:fixed_joint name="front_caster_adapter_to_front_caster_wheel" parent="front_caster_adapter" child="front_caster_wheel"
                        origin_position="0 0 -0.035"/>
-    <xacro:ball_link name="back_caster_wheel" mass="0.010" radius="0.015" use_collision="true"/>
+    <xacro:ball_link name="back_caster_wheel" mass="0.010" radius="0.015" friction="0.01" use_collision="true"/>
     <xacro:fixed_joint name="back_caster_adapter_to_back_caster_wheel" parent="back_caster_adapter" child="back_caster_wheel"
                        origin_position="0 0 -0.035"/>
